File: cq352_adapter.sch (KiCad schematic (older format))
At the start: 2 parts, among them J1 FSI-150, X1 CQ352_SOCKET

Commit message: connector layout
Parts:
- added J2, J3, J4: FSI-150, spels:FSI-150-10-L-D-M-AD, symbol spels:FSI-150
- X1: symbol spels_dev:CQ352_SOCKET -> cq352_adapter-rescue:CQ352_SOCKET-spels_dev
Connections:
- no-connect marks 0 -> 50
Other:
- moved on the sheet: J1A, J1B, J1C, J1D, J1E, X1A, X1B, X1C, X1D

Commit message: routing signals
Connections:
- net 93: now reaches J2.11
- net 93: now also X1.93
- net 95: now reaches J2.13
- net 95: now also X1.95
- net 97: now reaches J2.15
- net 97: now also X1.97
- net 99: now reaches J2.17
- net 99: now also X1.99
- net 101: now reaches J2.19
- net 101: now also X1.101
- net 103: now reaches J2.21
- net 103: now also X1.103
- net 105: now reaches J2.23
- net 105: now also X1.105
- net 107: now reaches J2.25
- net 107: now also X1.107
- net 109: now reaches J2.27
- net 109: now also X1.109
- net 111: now reaches J2.29
- net 111: now also X1.111
- net 113: now reaches J2.31
- net 113: now also X1.113
- net 115: now reaches J2.33
- net 115: now also X1.115
- net 117: now reaches J2.35
- net 117: now also X1.117
- net 119: now reaches J2.37
- net 119: now also X1.119
- net 121: now reaches J2.39
- net 121: now also X1.121
- net 123: now reaches J2.41
- net 123: now also X1.123
- net 125: now reaches J2.43
- net 125: now also X1.125
- net 127: now reaches J2.45
- net 127: now also X1.127
- net 129: now reaches J2.47
- net 129: now also X1.129
- net 131: now reaches J2.49
- net 131: now also X1.131
- net 89: now reaches J2.7
- net 89: now also X1.89
- net 91: now reaches J2.9
- net 91: now also X1.91
- net 92: now reaches J2.10
- net 92: now also X1.92
- net 94: now reaches J2.12
- net 94: now also X1.94
- net 96: now reaches J2.14
- net 96: now also X1.96
- net 98: now reaches J2.16
- net 98: now also X1.98
- net 100: now reaches J2.18
- net 100: now also X1.100
- net 102: now reaches J2.20
- net 102: now also X1.102
- net 104: now reaches J2.22
- net 104: now also X1.104
- net 106: now reaches J2.24
- net 106: now also X1.106
- net 108: now reaches J2.26
- net 108: now also X1.108
- net 110: now reaches J2.28
- net 110: now also X1.110
- net 112: now reaches J2.30
- net 112: now also X1.112
- net 114: now reaches J2.32
- net 114: now also X1.114
- net 116: now reaches J2.34
- net 116: now also X1.116
- net 118: now reaches J2.36
- net 118: now also X1.118
- net 120: now reaches J2.38
- net 120: now also X1.120
- net 122: now reaches J2.40
- net 122: now also X1.122
- net 124: now reaches J2.42
- net 124: now also X1.124
- net 126: now reaches J2.44
- net 126: now also X1.126
- net 128: now reaches J2.46
- net 128: now also X1.128
- net 130: now reaches J2.48
- net 130: now also X1.130
- net 132: now reaches J2.50
- net 132: now also X1.132
- net 90: now reaches J2.8
- net 90: now also X1.90
- net 133: now reaches J2.51
- net 133: now also X1.133
- net 135: now reaches J2.53
- net 135: now also X1.135
- net 137: now reaches J2.55
- net 137: now also X1.137
- net 139: now reaches J2.57
- net 139: now also X1.139
- net 141: now reaches J2.59
- net 141: now also X1.141
- net 143: now reaches J2.61
- net 143: now also X1.143
- net 145: now reaches J2.63
- net 145: now also X1.145
- net 147: now reaches J2.65
- net 147: now also X1.147
- net 149: now reaches J2.67
- net 149: now also X1.149
- net 151: now reaches J2.69
- net 151: now also X1.151
- net 153: now reaches J2.71
- net 153: now also X1.153
- net 155: now reaches J2.73
- net 155: now also X1.155
- net 157: now reaches J2.75
- net 157: now also X1.157
- net 159: now reaches J2.77
- net 159: now also X1.159
- net 161: now reaches J2.79
- net 161: now also X1.161
- net 163: now reaches J2.81
- net 163: now also X1.163
- net 165: now reaches J2.83
- net 165: now also X1.165
- net 167: now reaches J2.85
- net 167: now also X1.167
- net 169: now reaches J2.87
- net 169: now also X1.169
- net 171: now reaches J2.89
- net 171: now also X1.171
- net 173: now reaches J2.91
- net 173: now also X1.173
- net 175: now reaches J2.93
- net 175: now also X1.175
- net 134: now reaches J2.52
- net 134: now also X1.134
- net 136: now reaches J2.54
- net 136: now also X1.136
- net 138: now reaches J2.56
- net 138: now also X1.138
- net 140: now reaches J2.58
- net 140: now also X1.140
- net 142: now reaches J2.60
- net 142: now also X1.142
- net 144: now reaches J2.62
- net 144: now also X1.144
- net 146: now reaches J2.64
- net 146: now also X1.146
- net 148: now reaches J2.66
- net 148: now also X1.148
- net 150: now reaches J2.68
- net 150: now also X1.150
- net 152: now reaches J2.70
- net 152: now also X1.152
- net 154: now reaches J2.72
- net 154: now also X1.154
- net 156: now reaches J2.74
- net 156: now also X1.156
- net 158: now reaches J2.76
- net 158: now also X1.158
- net 160: now reaches J2.78
- net 160: now also X1.160
- net 162: now reaches J2.80
- net 162: now also X1.162
- net 164: now reaches J2.82
- net 164: now also X1.164
- net 166: now reaches J2.84
- net 166: now also X1.166
- net 168: now reaches J2.86
- net 168: now also X1.168
- net 170: now reaches J2.88
- net 170: now also X1.170
- net 172: now reaches J2.90
- net 172: now also X1.172
- net 174: now reaches J2.92
- net 174: now also X1.174
- net 176: now reaches J2.94
- net 176: now also X1.176
- net 1: now reaches X1.1
- net 1: now also J1.7
- net 10: now reaches X1.10
- net 10: now also J1.16
- net 11: now reaches X1.11
- net 11: now also J1.17
- net 12: now reaches X1.12
- net 12: now also J1.18
- net 13: now reaches X1.13
- net 13: now also J1.19
- net 14: now reaches X1.14
- net 14: now also J1.20
- net 15: now reaches X1.15
- net 15: now also J1.21
- net 16: now reaches X1.16
- net 16: now also J1.22
- net 17: now reaches X1.17
- net 17: now also J1.23
- net 18: now reaches X1.18
- net 18: now also J1.24
- net 19: now reaches X1.19
- net 19: now also J1.25
- net 2: now reaches X1.2
- net 2: now also J1.8
- net 20: now reaches X1.20
- net 20: now also J1.26
- net 21: now reaches X1.21
- net 21: now also J1.27
- net 22: now reaches X1.22
- net 22: now also J1.28
- net 23: now reaches X1.23
- net 23: now also J1.29
- net 24: now reaches X1.24
- net 24: now also J1.30
- net 25: now reaches X1.25
- net 25: now also J1.31
- net 26: now reaches X1.26
- net 26: now also J1.32
- net 27: now reaches X1.27
- net 27: now also J1.33
- net 28: now reaches X1.28
- net 28: now also J1.34
- net 29: now reaches X1.29
- net 29: now also J1.35
- net 3: now reaches X1.3
- net 3: now also J1.9
- net 30: now reaches X1.30
- net 30: now also J1.36
- net 31: now reaches X1.31
- net 31: now also J1.37
- net 32: now reaches X1.32
- net 32: now also J1.38
- net 33: now reaches X1.33
- net 33: now also J1.39
- net 34: now reaches X1.34
- net 34: now also J1.40
- net 35: now reaches X1.35
- net 35: now also J1.41
- net 36: now reaches X1.36
- net 36: now also J1.42
- net 37: now reaches X1.37
- net 37: now also J1.43
- net 38: now reaches X1.38
- net 38: now also J1.44
- net 39: now reaches X1.39
- net 39: now also J1.45
- net 4: now reaches X1.4
- net 4: now also J1.10
- net 40: now reaches X1.40
- net 40: now also J1.46
- net 41: now reaches X1.41
- net 41: now also J1.47
- net 42: now reaches X1.42
- net 42: now also J1.48
- net 43: now reaches X1.43
- net 43: now also J1.49
- net 44: now reaches X1.44
- net 44: now also J1.50
- net 45: now reaches X1.45
- net 45: now also J1.51
- net 46: now reaches X1.46
- net 46: now also J1.52
- net 47: now reaches X1.47
- net 47: now also J1.53
- net 48: now reaches X1.48
- net 48: now also J1.54
- net 49: now reaches X1.49
- net 49: now also J1.55
- net 5: now reaches X1.5
- net 5: now also J1.11
- net 50: now reaches X1.50
- net 50: now also J1.56
- net 51: now reaches X1.51
- net 51: now also J1.57
- net 52: now reaches X1.52
- net 52: now also J1.58
- net 53: now reaches X1.53
- net 53: now also J1.59
- net 54: now reaches X1.54
- net 54: now also J1.60
- net 55: now reaches X1.55
- net 55: now also J1.61
- net 56: now reaches X1.56
- net 56: now also J1.62
- net 57: now reaches X1.57
- net 57: now also J1.63
- net 58: now reaches X1.58
- net 58: now also J1.64
- net 59: now reaches X1.59
- net 59: now also J1.65
- net 6: now reaches X1.6
- net 6: now also J1.12
- net 60: now reaches X1.60
- net 60: now also J1.66
- net 61: now reaches X1.61
- net 61: now also J1.67
- net 62: now reaches X1.62
- net 62: now also J1.68
- net 63: now reaches X1.63
- net 63: now also J1.69
- net 64: now reaches X1.64
- net 64: now also J1.70
- net 65: now reaches X1.65
- net 65: now also J1.71
- net 66: now reaches X1.66
- net 66: now also J1.72
- net 67: now reaches X1.67
- net 67: now also J1.73
- net 68: now reaches X1.68
- net 68: now also J1.74
- net 69: now reaches X1.69
- net 69: now also J1.75
- net 7: now reaches X1.7
- net 7: now also J1.13
- net 70: now reaches X1.70
- net 70: now also J1.76
- net 71: now reaches X1.71
- net 71: now also J1.77
- net 72: now reaches X1.72
- net 72: now also J1.78
- net 73: now reaches X1.73
- net 73: now also J1.79
- net 74: now reaches X1.74
- net 74: now also J1.80
- net 75: now reaches X1.75
- net 75: now also J1.81
- net 76: now reaches X1.76
- net 76: now also J1.82
- net 77: now reaches X1.77
- net 77: now also J1.83
- net 78: now reaches X1.78
- net 78: now also J1.84
- net 79: now reaches X1.79
- net 79: now also J1.85
- net 8: now reaches X1.8
- net 8: now also J1.14
- net 80: now reaches X1.80
- net 80: now also J1.86
- net 81: now reaches X1.81
- net 81: now also J1.87
- net 82: now reaches X1.82
- net 82: now also J1.88
- net 83: now reaches X1.83
- net 83: now also J1.89
- net 84: now reaches X1.84
- net 84: now also J1.90
- net 85: now reaches X1.85
- net 85: now also J1.91
- net 86: now reaches X1.86
- net 86: now also J1.92
- net 87: now reaches X1.87
- net 87: now also J1.93
- net 88: now reaches X1.88
- net 88: now also J1.94
- net 9: now reaches X1.9
- net 9: now also J1.15
- net 177: now reaches X1.177
- net 177: now also J3.7
- net 178: now reaches X1.178
- net 178: now also J3.8
- net 179: now reaches X1.179
- net 179: now also J3.9
- net 180: now reaches X1.180
- net 180: now also J3.10
- net 181: now reaches X1.181
- net 181: now also J3.11
- net 182: now reaches X1.182
- net 182: now also J3.12
- net 183: now reaches X1.183
- net 183: now also J3.13
- net 184: now reaches X1.184
- net 184: now also J3.14
- net 185: now reaches X1.185
- net 185: now also J3.15
- net 186: now reaches X1.186
- net 186: now also J3.16
- net 187: now reaches X1.187
- net 187: now also J3.17
- net 188: now reaches X1.188
- net 188: now also J3.18
- net 189: now reaches X1.189
- net 189: now also J3.19
- net 190: now reaches X1.190
- net 190: now also J3.20
- net 191: now reaches X1.191
- net 191: now also J3.21
- net 192: now reaches X1.192
- net 192: now also J3.22
- net 193: now reaches X1.193
- net 193: now also J3.23
- net 194: now reaches X1.194
- net 194: now also J3.24
- net 195: now reaches X1.195
- net 195: now also J3.25
- net 196: now reaches X1.196
- net 196: now also J3.26
- net 197: now reaches X1.197
- net 197: now also J3.27
- net 198: now reaches X1.198
- net 198: now also J3.28
- net 199: now reaches X1.199
- net 199: now also J3.29
- net 200: now reaches X1.200
- net 200: now also J3.30
- net 201: now reaches X1.201
- net 201: now also J3.31
- net 202: now reaches X1.202
- net 202: now also J3.32
- net 203: now reaches X1.203
- net 203: now also J3.33
- net 204: now reaches X1.204
- net 204: now also J3.34
- net 205: now reaches X1.205
- net 205: now also J3.35
- net 206: now reaches X1.206
- net 206: now also J3.36
- net 207: now reaches X1.207
- net 207: now also J3.37
- net 208: now reaches X1.208
- net 208: now also J3.38
- net 209: now reaches X1.209
- net 209: now also J3.39
- net 210: now reaches X1.210
- net 210: now also J3.40
- net 211: now reaches X1.211
- net 211: now also J3.41
- net 212: now reaches X1.212
- net 212: now also J3.42
- net 213: now reaches X1.213
- net 213: now also J3.43
- net 214: now reaches X1.214
- net 214: now also J3.44
- net 215: now reaches X1.215
- net 215: now also J3.45
- net 216: now reaches X1.216
- net 216: now also J3.46
- net 217: now reaches X1.217
- net 217: now also J3.47
- net 218: now reaches X1.218
- net 218: now also J3.48
- net 219: now reaches X1.219
- net 219: now also J3.49
- net 220: now reaches X1.220
- net 220: now also J3.50
- net 221: now reaches X1.221
- net 221: now also J3.51
- net 222: now reaches X1.222
- net 222: now also J3.52
- net 223: now reaches X1.223
- net 223: now also J3.53
- net 224: now reaches X1.224
- net 224: now also J3.54
- net 225: now reaches X1.225
- net 225: now also J3.55
- net 226: now reaches X1.226
- net 226: now also J3.56
- net 227: now reaches X1.227
- net 227: now also J3.57
- net 228: now reaches X1.228
- net 228: now also J3.58
- net 229: now reaches X1.229
- net 229: now also J3.59
- net 230: now reaches X1.230
- net 230: now also J3.60
- net 231: now reaches X1.231
- net 231: now also J3.61
- net 232: now reaches X1.232
- net 232: now also J3.62
- net 233: now reaches X1.233
- net 233: now also J3.63
- net 234: now reaches X1.234
- net 234: now also J3.64
- net 235: now reaches X1.235
- net 235: now also J3.65
- net 236: now reaches X1.236
- net 236: now also J3.66
- net 237: now reaches X1.237
- net 237: now also J3.67
- net 238: now reaches X1.238
- net 238: now also J3.68
- net 239: now reaches X1.239
- net 239: now also J3.69
- net 240: now reaches X1.240
- net 240: now also J3.70
- net 241: now reaches X1.241
- net 241: now also J3.71
- net 242: now reaches X1.242
- net 242: now also J3.72
- net 243: now reaches X1.243
- net 243: now also J3.73
- net 244: now reaches X1.244
- net 244: now also J3.74
- net 245: now reaches X1.245
- net 245: now also J3.75
- net 246: now reaches X1.246
- net 246: now also J3.76
- net 247: now reaches X1.247
- net 247: now also J3.77
- net 248: now reaches X1.248
- net 248: now also J3.78
- net 249: now reaches X1.249
- net 249: now also J3.79
- net 250: now reaches X1.250
- net 250: now also J3.80
- net 251: now reaches X1.251
- net 251: now also J3.81
- net 252: now reaches X1.252
- net 252: now also J3.82
- net 253: now reaches X1.253
- net 253: now also J3.83
- net 254: now reaches X1.254
- net 254: now also J3.84
- net 255: now reaches X1.255
- net 255: now also J3.85
- net 256: now reaches X1.256
- net 256: now also J3.86
- net 257: now reaches X1.257
- net 257: now also J3.87
- net 258: now reaches X1.258
- net 258: now also J3.88
- net 259: now reaches X1.259
- net 259: now also J3.89
- net 260: now reaches X1.260
- net 260: now also J3.90
- net 261: now reaches X1.261
- net 261: now also J3.91
- net 262: now reaches X1.262
- net 262: now also J3.92
- net 263: now reaches X1.263
- net 263: now also J3.93
- net 264: now reaches X1.264
- net 264: now also J3.94
- net 265: now reaches X1.265
- net 265: now also J4.7
- net 266: now reaches X1.266
- net 266: now also J4.8
- net 267: now reaches X1.267
- net 267: now also J4.9
- net 268: now reaches X1.268
- net 268: now also J4.10
- net 269: now reaches X1.269
- net 269: now also J4.11
- net 270: now reaches X1.270
- net 270: now also J4.12
- net 271: now reaches X1.271
- net 271: now also J4.13
- net 272: now reaches X1.272
- net 272: now also J4.14
- net 273: now reaches X1.273
- net 273: now also J4.15
- net 274: now reaches X1.274
- net 274: now also J4.16
- net 275: now reaches X1.275
- net 275: now also J4.17
- net 276: now reaches X1.276
- net 276: now also J4.18
- net 277: now reaches X1.277
- net 277: now also J4.19
- net 278: now reaches X1.278
- net 278: now also J4.20
- net 279: now reaches X1.279
- net 279: now also J4.21
- net 280: now reaches X1.280
- net 280: now also J4.22
- net 281: now reaches X1.281
- net 281: now also J4.23
- net 282: now reaches X1.282
- net 282: now also J4.24
- net 283: now reaches X1.283
- net 283: now also J4.25
- net 284: now reaches X1.284
- net 284: now also J4.26
- net 285: now reaches X1.285
- net 285: now also J4.27
- net 286: now reaches X1.286
- net 286: now also J4.28
- net 287: now reaches X1.287
- net 287: now also J4.29
- net 288: now reaches X1.288
- net 288: now also J4.30
- net 289: now reaches X1.289
- net 289: now also J4.31
- net 290: now reaches X1.290
- net 290: now also J4.32
- net 291: now reaches X1.291
- net 291: now also J4.33
- net 292: now reaches X1.292
- net 292: now also J4.34
- net 293: now reaches X1.293
- net 293: now also J4.35
- net 294: now reaches X1.294
- net 294: now also J4.36
- net 295: now reaches X1.295
- net 295: now also J4.37
- net 296: now reaches X1.296
- net 296: now also J4.38
- net 297: now reaches X1.297
- net 297: now also J4.39
- net 298: now reaches X1.298
- net 298: now also J4.40
- net 299: now reaches X1.299
- net 299: now also J4.41
- net 300: now reaches X1.300
- net 300: now also J4.42
- net 301: now reaches X1.301
- net 301: now also J4.43
- net 302: now reaches X1.302
- net 302: now also J4.44
- net 303: now reaches X1.303
- net 303: now also J4.45
- net 304: now reaches X1.304
- net 304: now also J4.46
- net 305: now reaches X1.305
- net 305: now also J4.47
- net 306: now reaches X1.306
- net 306: now also J4.48
- net 307: now reaches X1.307
- net 307: now also J4.49
- net 308: now reaches X1.308
- net 308: now also J4.50
- net 309: now reaches X1.309
- net 309: now also J4.51
- net 310: now reaches X1.310
- net 310: now also J4.52
- net 311: now reaches X1.311
- net 311: now also J4.53
- net 312: now reaches X1.312
- net 312: now also J4.54
- net 313: now reaches X1.313
- net 313: now also J4.55
- net 314: now reaches X1.314
- net 314: now also J4.56
- net 315: now reaches X1.315
- net 315: now also J4.57
- net 316: now reaches X1.316
- net 316: now also J4.58
- net 317: now reaches X1.317
- net 317: now also J4.59
- net 318: now reaches X1.318
- net 318: now also J4.60
- net 319: now reaches X1.319
- net 319: now also J4.61
- net 320: now reaches X1.320
- net 320: now also J4.62
- net 321: now reaches X1.321
- net 321: now also J4.63
- net 322: now reaches X1.322
- net 322: now also J4.64
- net 323: now reaches X1.323
- net 323: now also J4.65
- net 324: now reaches X1.324
- net 324: now also J4.66
- net 325: now reaches X1.325
- net 325: now also J4.67
- net 326: now reaches X1.326
- net 326: now also J4.68
- net 327: now reaches X1.327
- net 327: now also J4.69
- net 328: now reaches X1.328
- net 328: now also J4.70
- net 329: now reaches X1.329
- net 329: now also J4.71
- net 330: now reaches X1.330
- net 330: now also J4.72
- net 331: now reaches X1.331
- net 331: now also J4.73
- net 332: now reaches X1.332
- net 332: now also J4.74
- net 333: now reaches X1.333
- net 333: now also J4.75
- net 334: now reaches X1.334
- net 334: now also J4.76
- net 335: now reaches X1.335
- net 335: now also J4.77
- net 336: now reaches X1.336
- net 336: now also J4.78
- net 337: now reaches X1.337
- net 337: now also J4.79
- net 338: now reaches X1.338
- net 338: now also J4.80
- net 339: now reaches X1.339
- net 339: now also J4.81
- net 340: now reaches X1.340
- net 340: now also J4.82
- net 341: now reaches X1.341
- net 341: now also J4.83
- net 342: now reaches X1.342
- net 342: now also J4.84
- net 343: now reaches X1.343
- net 343: now also J4.85
- net 344: now reaches X1.344
- net 344: now also J4.86
- net 345: now reaches X1.345
- net 345: now also J4.87
- net 346: now reaches X1.346
- net 346: now also J4.88
- net 347: now reaches X1.347
- net 347: now also J4.89
- net 348: now reaches X1.348
- net 348: now also J4.90
- net 349: now reaches X1.349
- net 349: now also J4.91
- net 350: now reaches X1.350
- net 350: now also J4.92
- net 351: now reaches X1.351
- net 351: now also J4.93
- net 352: now reaches X1.352
- net 352: now also J4.94
- no-connect marks 50 -> 61
Other:
- moved on the sheet: X1A
